File: pcb/midimerger/midimerger.sch (KiCad schematic (older format))
At the start: 11 parts, among them J1 USB_A, J2 MIDI_1_IN, J3 MIDI_1_OUT, U1 Teensy3.6, U2 6N138

Commit message: Added digikey
Parts:
- C1: footprint (none) -> Capacitor_THT:CP_Radial_D4.0mm_P2.00mm
- J1: footprint (none) -> digikey-footprints:USB_A_Female_UE27AC54100
- J2, J3: footprint (none) -> Eurocad:MIDI_DIN5
- U1: footprint teensy:Teensy1.0 -> teensy:Teensy35_36
Changed lines of the file:
@@
 EESchema Schematic File Version 4
+LIBS:midimerger-cache
 EELAYER 26 0
 EELAYER END
@@
 F 0 "U1" H 3150 6337 60  0000 C CNN
 F 1 "Teensy3.6" H 3150 6231 60  0000 C CNN
-F 2 "teensy:Teensy1.0" H 2900 3950 60  0001 C CNN
+F 2 "teensy:Teensy35_36" H 2900 3950 60  0001 C CNN
 F 3 "" H 2900 3950 60  0000 C CNN
 	1    3150 3950
@@
 F 0 "J1" H 7205 2517 50  0000 C CNN
 F 1 "USB_A" H 7205 2426 50  0000 C CNN
-F 2 "" H 7300 2000 50  0001 C CNN
+F 2 "digikey-footprints:USB_A_Female_UE27AC54100" H 7300 2000 50  0001 C CNN
 F 3 " ~" H 7300 2000 50  0001 C CNN
 	1    7150 2050
@@
 F 0 "J2" H 6550 2883 50  0000 C CNN
 F 1 "MIDI_1_IN" H 6550 2974 50  0000 C CNN
-F 2 "" H 6550 3250 50  0001 C CNN
+F 2 "Eurocad:MIDI_DIN5" H 6550 3250 50  0001 C CNN
 F 3 "http://www.mouser.com/ds/2/18/40_c091_abd_e-75918.pdf" H 6550 3250 50  0001 C CNN
 	1    6550 3250
@@
 F 0 "J3" H 7600 2833 50  0000 C CNN
 F 1 "MIDI_1_OUT" H 7600 2924 50  0000 C CNN
-F 2 "" H 7600 3200 50  0001 C CNN
+F 2 "Eurocad:MIDI_DIN5" H 7600 3200 50  0001 C CNN
 F 3 "http://www.mouser.com/ds/2/18/40_c091_abd_e-75918.pdf" H 7600 3200 50  0001 C CNN
 	1    7600 3200
@@
 F 0 "C1" V 7278 5000 50  0000 C CNN
 F 1 "0.1uf" V 7187 5000 50  0000 C CNN
-F 2 "" H 7050 5000 50  0001 C CNN
+F 2 "Capacitor_THT:CP_Radial_D4.0mm_P2.00mm" H 7050 5000 50  0001 C CNN
 F 3 "~" H 7050 5000 50  0001 C CNN
 	1    7050 5000

Commit message: updated pcb
Parts:
- U1: symbol teensy:Teensy3.6 -> midimerger-rescue:Teensy3.6-teensy
Changed lines of the file:
@@
 $EndDescr
 $Comp
-L teensy:Teensy3.6 U1
+L midimerger-rescue:Teensy3.6-teensy U1
 U 1 1 5C3FEA3C
 P 3150 3950
@@
 Wire Wire Line
 	6450 5300 6450 5600
+$Comp
+L power:GND #PWR?
+U 1 1 5C4457FD
+P 1950 4450
+F 0 "#PWR?" H 1950 4200 50  0001 C CNN
+F 1 "GND" V 1955 4322 50  0000 R CNN
+F 2 "" H 1950 4450 50  0001 C CNN
+F 3 "" H 1950 4450 50  0001 C CNN
+	1    1950 4450
+	0    1    1    0
+$EndComp
+$Comp
+L power:GND #PWR?
+U 1 1 5C4463B2
+P -9100 -4000
+F 0 "#PWR?" H -9100 -4250 50  0001 C CNN
+F 1 "GND" V -9095 -4128 50  0000 R CNN
+F 2 "" H -9100 -4000 50  0001 C CNN
+F 3 "" H -9100 -4000 50  0001 C CNN
+	1    -9100 -4000
+	0    -1   -1   0
+$EndComp
 $EndSCHEMATC

Commit message: added export
Parts:
- R1, R2, R3, R4: footprint Resistor_THT:R_Axial_DIN0309_L9.0mm_D3.2mm_P15.24mm_Horizontal -> Resistor_THT:R_Axial_DIN0309_L9.0mm_D3.2mm_P12.70mm_Horizontal
Changed lines of the file:
@@
 F 0 "R3" H 7970 3496 50  0000 L CNN
 F 1 "220" H 7970 3405 50  0000 L CNN
-F 2 "Resistor_THT:R_Axial_DIN0309_L9.0mm_D3.2mm_P15.24mm_Horizontal" V 7830 3450 50  0001 C CNN
+F 2 "Resistor_THT:R_Axial_DIN0309_L9.0mm_D3.2mm_P12.70mm_Horizontal" V 7830 3450 50  0001 C CNN
 F 3 "~" H 7900 3450 50  0001 C CNN
 	1    7900 3450
@@
 F 0 "R1" H 6920 3796 50  0000 L CNN
 F 1 "220" H 6920 3705 50  0000 L CNN
-F 2 "Resistor_THT:R_Axial_DIN0309_L9.0mm_D3.2mm_P15.24mm_Horizontal" V 6780 3750 50  0001 C CNN
+F 2 "Resistor_THT:R_Axial_DIN0309_L9.0mm_D3.2mm_P12.70mm_Horizontal" V 6780 3750 50  0001 C CNN
 F 3 "~" H 6850 3750 50  0001 C CNN
 	1    6850 3750
@@
 F 0 "R2" H 7370 3946 50  0000 L CNN
 F 1 "220" H 7370 3855 50  0000 L CNN
-F 2 "Resistor_THT:R_Axial_DIN0309_L9.0mm_D3.2mm_P15.24mm_Horizontal" V 7230 3900 50  0001 C CNN
+F 2 "Resistor_THT:R_Axial_DIN0309_L9.0mm_D3.2mm_P12.70mm_Horizontal" V 7230 3900 50  0001 C CNN
 F 3 "~" H 7300 3900 50  0001 C CNN
 	1    7300 3900
@@
 F 0 "R4" V 6807 5300 50  0000 C CNN
 F 1 "470" V 6716 5300 50  0000 C CNN
-F 2 "Resistor_THT:R_Axial_DIN0309_L9.0mm_D3.2mm_P15.24mm_Horizontal" V 6530 5300 50  0001 C CNN
+F 2 "Resistor_THT:R_Axial_DIN0309_L9.0mm_D3.2mm_P12.70mm_Horizontal" V 6530 5300 50  0001 C CNN
 F 3 "~" H 6600 5300 50  0001 C CNN
 	1    6600 5300
@@
 	6450 5300 6450 5600
 $Comp
-L power:GND #PWR?
+L power:GND #PWR0107
 U 1 1 5C4457FD
 P 1950 4450
-F 0 "#PWR?" H 1950 4200 50  0001 C CNN
+F 0 "#PWR0107" H 1950 4200 50  0001 C CNN
 F 1 "GND" V 1955 4322 50  0000 R CNN
 F 2 "" H 1950 4450 50  0001 C CNN
@@
 $EndComp
 $Comp
-L power:GND #PWR?
+L power:GND #PWR0108
 U 1 1 5C4463B2
 P -9100 -4000
-F 0 "#PWR?" H -9100 -4250 50  0001 C CNN
+F 0 "#PWR0108" H -9100 -4250 50  0001 C CNN
 F 1 "GND" V -9095 -4128 50  0000 R CNN
 F 2 "" H -9100 -4000 50  0001 C CNN

Commit message: updated pcb
Connections:
- wire segments 47 -> 49
Changed lines of the file:
@@
 Connection ~ 7050 2550
-Wire Wire Line
-	7050 2550 7050 2600
 Wire Wire Line
 	7450 2150 7800 2150
@@
 L power:GND #PWR0107
 U 1 1 5C4457FD
-P 1950 4450
-F 0 "#PWR0107" H 1950 4200 50  0001 C CNN
-F 1 "GND" V 1955 4322 50  0000 R CNN
-F 2 "" H 1950 4450 50  0001 C CNN
-F 3 "" H 1950 4450 50  0001 C CNN
-	1    1950 4450
+P 1800 4250
+F 0 "#PWR0107" H 1800 4000 50  0001 C CNN
+F 1 "GND" V 1805 4122 50  0000 R CNN
+F 2 "" H 1800 4250 50  0001 C CNN
+F 3 "" H 1800 4250 50  0001 C CNN
+	1    1800 4250
 	0    1    1    0
 $EndComp
@@
 	0    -1   -1   0
 $EndComp
+Wire Wire Line
+	1800 4250 1800 4450
+Wire Wire Line
+	1800 4450 1950 4450
+$Comp
+L power:GND #PWR?
+U 1 1 5C4BFF93
+P 7050 2750
+F 0 "#PWR?" H 7050 2500 50  0001 C CNN
+F 1 "GND" H 7055 2577 50  0000 C CNN
+F 2 "" H 7050 2750 50  0001 C CNN
+F 3 "" H 7050 2750 50  0001 C CNN
+	1    7050 2750
+	1    0    0    -1
+$EndComp
+Wire Wire Line
+	7050 2550 7050 2750
 $EndSCHEMATC

Commit message: update schematics
Connections:
- net labels added: 3.3V
- wire segments 49 -> 50
Changed lines of the file:
@@
 Wire Wire Line
 	6750 4950 6750 5000
-Text Label 6750 5150 0    50   ~ 0
+Text Label 7000 5200 0    50   ~ 0
 5V
 $Comp
@@
 Wire Wire Line
 	6350 4950 6350 5100
-Wire Wire Line
-	6750 5000 6750 5300
 Text Label 1600 1950 0    50   ~ 0
 MIDI_1_IN
@@
 Text Label 7300 4250 0    50   ~ 0
 MIDI_1_OUT
-Connection ~ 6750 5000
 Wire Wire Line
 	6450 4950 6450 5300
@@
 	1800 4450 1950 4450
 $Comp
-L power:GND #PWR?
+L power:GND #PWR0109
 U 1 1 5C4BFF93
 P 7050 2750
-F 0 "#PWR?" H 7050 2500 50  0001 C CNN
+F 0 "#PWR0109" H 7050 2500 50  0001 C CNN
 F 1 "GND" H 7055 2577 50  0000 C CNN
 F 2 "" H 7050 2750 50  0001 C CNN
@@
 Wire Wire Line
 	7050 2550 7050 2750
+Wire Wire Line
+	4350 5350 4700 5350
+Text Label 4450 5350 0    50   ~ 0
+3.3V
+Wire Wire Line
+	6750 5300 7000 5300
+Text Label 6850 5300 3    50   ~ 0
+3.3V
 $EndSCHEMATC

Commit message: fixed 5v
Parts:
- U1: symbol midimerger-rescue:Teensy3.6-teensy -> midimerger-rescue:Teensy3.6-teensy-midimerger-rescue
Connections:
- wire segments 50 -> 53
Changed lines of the file:
@@
 $EndDescr
 $Comp
-L midimerger-rescue:Teensy3.6-teensy U1
+L midimerger-rescue:Teensy3.6-teensy-midimerger-rescue U1
 U 1 1 5C3FEA3C
 P 3150 3950
@@
 $EndComp
 Wire Wire Line
-	6750 5000 6950 5000
+	6750 5000 6850 5000
 Wire Wire Line
 	7150 5000 7200 5000
@@
 Wire Wire Line
 	6750 5300 7000 5300
-Text Label 6850 5300 3    50   ~ 0
+Text Label 7000 5300 0    50   ~ 0
 3.3V
+Wire Wire Line
+	7000 5200 6850 5200
+Wire Wire Line
+	6850 5200 6850 5000
+Connection ~ 6850 5000
+Wire Wire Line
+	6850 5000 6950 5000
 $EndSCHEMATC
